File: motorplank.brd (EAGLE design)
At the start: 80 x 49 mm, 18 parts, among them IC1 74AHC1G86DBV

Commit message: Move capacitors to the side closer to ground.
Parts:
- moved C3 19.7 mm to (16.8, 14.9)
- moved C2 11.4 mm to (16.8, 18.7)
Routing:
- net VMOT: track 87.1 -> 86.1 mm
Changed lines of the file:
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@@
 <board>
 <plain>
-<text x="41.275" y="34.29" size="1.778" layer="21" align="bottom-center">Loki DC Motor Plank v0.1</text>
+<text x="41.275" y="34.29" size="1.778" layer="21" font="vector" align="bottom-center">Loki DC Motor Plank v0.1</text>
 <text x="75.8825" y="27.94" size="2.54" layer="21" align="bottom-center">+</text>
 <text x="75.8825" y="18.7325" size="2.54" layer="21" align="bottom-center">-</text>
-<text x="71.755" y="24.13" size="1.27" layer="21" rot="R90" align="bottom-center">DC in 6-20V</text>
-<text x="20.32" y="2.54" size="0.762" layer="21" align="bottom-center">Bridge SJ2 to connect VIN and external power</text>
+<text x="71.755" y="24.13" size="1.27" layer="21" font="vector" rot="R90" align="bottom-center">DC in 6-20V</text>
+<text x="20.32" y="2.54" size="0.762" layer="21" font="vector" align="bottom-center">Bridge SJ2 to connect VIN and external power</text>
 </plain>
 <attributes>
@@
 <element name="SJ2" library="jumper" package="SJ" value="" x="49.53" y="10.16" rot="R270"/>
 <element name="C1" library="SparkFun-Passives" package="0603-CAP" value="0.1u" x="23.8125" y="25.0825"/>
-<element name="C2" library="SparkFun-Passives" package="0603-CAP" value="0.1u" x="16.8275" y="30.1625" rot="R180"/>
-<element name="C3" library="SparkFun-Passives" package="PANASONIC_C" value="10u" x="16.8275" y="34.6075"/>
+<element name="C2" library="SparkFun-Passives" package="0603-CAP" value="0.1u" x="16.8275" y="18.7325" rot="R180"/>
+<element name="C3" library="SparkFun-Passives" package="PANASONIC_C" value="10u" x="16.8275" y="14.9225"/>
 <element name="U$4" library="SparkFun-Aesthetics" package="OSHW-LOGO-M" value="" x="41.275" y="4.445"/>
 <element name="U$5" library="nickparts" package="BILED" value="BILED" x="6.6675" y="35.8775"/>
@@
 <wire x1="14.605" y1="22.5425" x2="16.51" y2="22.5425" width="1.016" layer="16"/>
 <wire x1="14.605" y1="22.5425" x2="12.7" y2="22.5425" width="1.016" layer="1"/>
-<wire x1="15.0275" y1="34.4075" x2="15.0275" y2="30.1625" width="1.016" layer="1"/>
-<wire x1="15.0275" y1="30.1625" x2="15.0275" y2="26.775" width="1.016" layer="1"/>
-<wire x1="15.0275" y1="26.775" x2="14.605" y2="26.3525" width="1.016" layer="1"/>
-<wire x1="15.9775" y1="30.1625" x2="15.0275" y2="30.1625" width="1.016" layer="1"/>
 <wire x1="16.51" y1="17.78" x2="16.8275" y2="17.4625" width="0.508" layer="16"/>
 <wire x1="20.4835" y1="24.1225" x2="24.447503125" y2="24.12818125" width="0.508" layer="1"/>
@@
 <vertex x="24.765" y="36.83"/>
 <vertex x="10.16" y="36.83"/>
-<vertex x="10.16" y="15.24"/>
-<vertex x="24.765" y="15.24"/>
+<vertex x="10.16" y="11.43"/>
+<vertex x="24.765" y="11.43"/>
 </polygon>
 <polygon width="0.508" layer="1" isolate="0.254">
-<vertex x="19.05" y="15.24"/>
-<vertex x="13.97" y="15.24"/>
+<vertex x="19.05" y="11.43"/>
+<vertex x="13.97" y="11.43"/>
 <vertex x="13.97" y="36.83"/>
 <vertex x="19.05" y="36.83"/>
 </polygon>
-<via x="16.8275" y="15.5575" extent="1-16" drill="0.5"/>
-<via x="16.8275" y="16.8275" extent="1-16" drill="0.5"/>
-<via x="16.8275" y="18.0975" extent="1-16" drill="0.5"/>
-<via x="16.8275" y="19.3675" extent="1-16" drill="0.5"/>
 <via x="16.8275" y="28.2575" extent="1-16" drill="0.5"/>
 <via x="16.8275" y="26.9875" extent="1-16" drill="0.5"/>
@@
 <wire x1="75.8825" y1="22.5425" x2="63.1825" y2="22.5425" width="1.016" layer="16"/>
 <wire x1="63.1825" y1="22.5425" x2="57.15" y2="16.51" width="1.016" layer="16"/>
+<wire x1="15.0275" y1="14.7225" x2="15.0275" y2="18.7325" width="1.016" layer="1"/>
+<wire x1="15.0275" y1="18.7325" x2="15.0275" y2="22.12" width="1.016" layer="1"/>
+<wire x1="15.0275" y1="22.12" x2="14.605" y2="22.5425" width="1.016" layer="1"/>
+<wire x1="15.9775" y1="18.7325" x2="15.0275" y2="18.7325" width="1.016" layer="1"/>
+<via x="16.8275" y="33.3375" extent="1-16" drill="0.5"/>
+<via x="16.8275" y="32.0675" extent="1-16" drill="0.5"/>
+<via x="16.8275" y="30.7975" extent="1-16" drill="0.5"/>
+<via x="16.8275" y="29.5275" extent="1-16" drill="0.5"/>
+<wire x1="16.8275" y1="28.2575" x2="16.8275" y2="29.5275" width="0" layer="19" extent="1-1"/>
 </signal>
 <signal name="A0">
@@
 <wire x1="51.1175" y1="22.5425" x2="49.53" y2="20.955" width="1.016" layer="1"/>
 <wire x1="19.05" y1="27.6225" x2="19.05" y2="21.2725" width="1.016" layer="1"/>
-<wire x1="19.05" y1="21.2725" x2="19.3675" y2="20.955" width="1.016" layer="1"/>
+<wire x1="19.05" y1="21.2725" x2="19.20875" y2="21.11375" width="1.016" layer="1"/>
+<wire x1="19.20875" y1="21.11375" x2="19.3675" y2="20.955" width="1.016" layer="1"/>
 <wire x1="19.3675" y1="20.955" x2="20.0025" y2="20.955" width="1.016" layer="1"/>
-<wire x1="19.45" y1="29.845" x2="19.45" y2="33.685" width="1.016" layer="1"/>
-<wire x1="19.45" y1="33.685" x2="18.7275" y2="34.4075" width="1.016" layer="1"/>
-<wire x1="17.6775" y1="30.1625" x2="19.05" y2="30.1625" width="1.016" layer="1"/>
-<wire x1="19.05" y1="30.1625" x2="19.1325" y2="30.1625" width="1.016" layer="1"/>
-<wire x1="19.1325" y1="30.1625" x2="19.45" y2="29.845" width="1.016" layer="1"/>
 <wire x1="20.4835" y1="21.5225" x2="20.4835" y2="20.8725" width="0.3048" layer="1"/>
 <wire x1="20.4025" y1="20.8725" x2="20.32" y2="20.955" width="0.3048" layer="1"/>
 <wire x1="19.05" y1="27.6225" x2="19.05" y2="28.2575" width="1.016" layer="1"/>
-<wire x1="19.05" y1="28.2575" x2="19.05" y2="30.1625" width="1.016" layer="1"/>
 <wire x1="20.4835" y1="28.0225" x2="19.285" y2="28.0225" width="0.508" layer="1"/>
 <wire x1="19.285" y1="28.0225" x2="19.05" y2="28.2575" width="0.508" layer="1"/>
@@
 <wire x1="75.8825" y1="26.0425" x2="54.6175" y2="26.0425" width="1.016" layer="1"/>
 <wire x1="54.6175" y1="26.0425" x2="51.1175" y2="22.5425" width="1.016" layer="1"/>
+<wire x1="18.7275" y1="14.7225" x2="18.7275" y2="18.7325" width="1.016" layer="1"/>
+<wire x1="18.7275" y1="18.7325" x2="18.7275" y2="20.6325" width="1.016" layer="1"/>
+<wire x1="18.7275" y1="20.6325" x2="19.20875" y2="21.11375" width="1.016" layer="1"/>
+<wire x1="17.6775" y1="18.7325" x2="18.7275" y2="18.7325" width="1.016" layer="1"/>
 </signal>
 <signal name="PWMA">
