File: displayplank.brd (EAGLE design)
At the start: 50 x 49 mm, 15 parts, among them Q1 MOSFET-NCHANNELSMD

Commit message: Replace usb mini connector with usb micro one.
Other:
- board text added: "Loki Display Plank v0.1"
- board text removed: "Display Plank v0.1"
Changed lines of the file:
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@@
 <board>
 <plain>
-<text x="25.4" y="46.355" size="2.032" layer="1" font="vector" align="bottom-center">Display Plank v0.1</text>
+<text x="25.4" y="46.355" size="2.032" layer="1" font="vector" align="bottom-center">Loki Display Plank v0.1</text>
 </plain>
 <attributes>
