File: schematics/displayplank/displayplank.sch (EAGLE design)
At the start: 14 parts, among them Q1 MOSFET-NCHANNELSMD

Commit message: Tweaks to planks; change 0604 parts for 0805 where possible
Also added 4 pin plank; minor text changes.
Parts:
- added C1, C2: 0.1u, SparkFun-Passives:CAP0805
- R1, R2, R3, R4: device SparkFun-Passives:RESISTOR0603-RES -> SparkFun-Passives:RESISTOR0805-RES
Connections:
- net +3V3: now also C1.1
- net +5V: now also C2.1
- net GND: now also C1.2, C2.2
Changed lines of the file:
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@@
 <part name="LED3" library="led" deviceset="LED" device="SML0805"/>
 <part name="LED4" library="led" deviceset="LED" device="SML0805"/>
-<part name="R1" library="SparkFun-Passives" deviceset="RESISTOR" device="0603-RES" value="340"/>
-<part name="R2" library="SparkFun-Passives" deviceset="RESISTOR" device="0603-RES" value="340"/>
-<part name="R3" library="SparkFun-Passives" deviceset="RESISTOR" device="0603-RES" value="340"/>
-<part name="R4" library="SparkFun-Passives" deviceset="RESISTOR" device="0603-RES" value="340"/>
+<part name="R1" library="SparkFun-Passives" deviceset="RESISTOR" device="0805-RES" value="340"/>
+<part name="R2" library="SparkFun-Passives" deviceset="RESISTOR" device="0805-RES" value="340"/>
+<part name="R3" library="SparkFun-Passives" deviceset="RESISTOR" device="0805-RES" value="340"/>
+<part name="R4" library="SparkFun-Passives" deviceset="RESISTOR" device="0805-RES" value="340"/>
 <part name="Q1" library="SparkFun-DiscreteSemi" deviceset="MOSFET-NCHANNEL" device="SMD"/>
 <part name="P+3" library="supply1" deviceset="+5V" device=""/>
@@
 <part name="U$3" library="nickparts" deviceset="JOYSTICK-10MM" device=""/>
 <part name="GND5" library="supply1" deviceset="GND" device=""/>
+<part name="C1" library="SparkFun-Passives" deviceset="CAP" device="0805" value="0.1u"/>
+<part name="+3V5" library="supply1" deviceset="+3V3" device=""/>
+<part name="GND6" library="supply1" deviceset="GND" device=""/>
+<part name="P+4" library="supply1" deviceset="+5V" device=""/>
+<part name="C2" library="SparkFun-Passives" deviceset="CAP" device="0805" value="0.1u"/>
+<part name="GND7" library="supply1" deviceset="GND" device=""/>
 </parts>
 <sheets>
@@
 <instance part="U$3" gate="G$1" x="27.94" y="-17.78"/>
 <instance part="GND5" gate="1" x="22.86" y="-27.94"/>
+<instance part="C1" gate="G$1" x="134.62" y="-45.72"/>
+<instance part="+3V5" gate="G$1" x="134.62" y="-38.1"/>
+<instance part="GND6" gate="1" x="134.62" y="-50.8"/>
+<instance part="P+4" gate="1" x="127" y="-38.1"/>
+<instance part="C2" gate="G$1" x="127" y="-45.72"/>
+<instance part="GND7" gate="1" x="127" y="-50.8"/>
 </instances>
 <busses>
@@
 <junction x="101.6" y="35.56"/>
 </segment>
+<segment>
+<pinref part="P+4" gate="1" pin="+5V"/>
+<pinref part="C2" gate="G$1" pin="1"/>
+</segment>
 </net>
 <net name="+3V3" class="0">
@@
 <wire x1="116.84" y1="-20.32" x2="114.3" y2="-20.32" width="0.1524" layer="91"/>
 <wire x1="114.3" y1="-20.32" x2="114.3" y2="-10.16" width="0.1524" layer="91"/>
+</segment>
+<segment>
+<pinref part="C1" gate="G$1" pin="1"/>
+<pinref part="+3V5" gate="G$1" pin="+3V3"/>
 </segment>
 </net>
@@
 <wire x1="22.86" y1="-22.86" x2="22.86" y2="-25.4" width="0.1524" layer="91"/>
 </segment>
+<segment>
+<pinref part="C1" gate="G$1" pin="2"/>
+<pinref part="GND6" gate="1" pin="GND"/>
+</segment>
+<segment>
+<pinref part="C2" gate="G$1" pin="2"/>
+<pinref part="GND7" gate="1" pin="GND"/>
+</segment>
 </net>

Commit message: Displayplank: Added pulldown for FET, improved capacitor spacing, fixed layer of name text.
Parts:
- added R5: 100k, SparkFun-Passives:RESISTOR0805-RES
Connections:
- net GND: now also R5.1
- net LIGHT: now also R5.2
Changed lines of the file:
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@@
 <part name="C2" library="SparkFun-Passives" deviceset="CAP" device="0805" value="0.1u"/>
 <part name="GND7" library="supply1" deviceset="GND" device=""/>
+<part name="R5" library="SparkFun-Passives" deviceset="RESISTOR" device="0805-RES" value="100k"/>
 </parts>
 <sheets>
@@
 <instance part="Q1" gate="G$1" x="96.52" y="10.16"/>
 <instance part="P+3" gate="1" x="96.52" y="40.64"/>
-<instance part="GND4" gate="1" x="96.52" y="0"/>
+<instance part="GND4" gate="1" x="96.52" y="-5.08"/>
 <instance part="U$5" gate="G$1" x="116.84" y="-25.4"/>
 <instance part="+3V4" gate="G$1" x="114.3" y="-7.62"/>
@@
 <instance part="C2" gate="G$1" x="127" y="-45.72"/>
 <instance part="GND7" gate="1" x="127" y="-50.8"/>
+<instance part="R5" gate="G$1" x="88.9" y="5.08" rot="R90"/>
 </instances>
 <busses>
@@
 <pinref part="Q1" gate="G$1" pin="S"/>
 <pinref part="GND4" gate="1" pin="GND"/>
-<wire x1="96.52" y1="5.08" x2="96.52" y2="2.54" width="0.1524" layer="91"/>
+<wire x1="96.52" y1="5.08" x2="96.52" y2="0" width="0.1524" layer="91"/>
+<pinref part="R5" gate="G$1" pin="1"/>
+<wire x1="96.52" y1="0" x2="96.52" y2="-2.54" width="0.1524" layer="91"/>
+<wire x1="88.9" y1="0" x2="96.52" y2="0" width="0.1524" layer="91"/>
+<junction x="96.52" y="0"/>
 </segment>
 <segment>
@@
 <wire x1="88.9" y1="10.16" x2="83.82" y2="10.16" width="0.1524" layer="91"/>
 <label x="81.28" y="10.16" size="1.778" layer="95"/>
-</segment>
-</net>
+<pinref part="R5" gate="G$1" pin="2"/>
+<junction x="88.9" y="10.16"/>
+</segment>
+</net>
