File: schematics/programmer/programmer.sch (EAGLE design)
At the start: 15 parts, among them CN1 M05X2-0.05-SMD, IC1 CY7C68013A-56PVXC, U2 TLV702XX, Y1 24MHz

Commit message: Fixed both Loki and the programmer to use 3.3v for power on programming headers.
Connections:
- net VBUS: no longer JP4.1
- net VCC: now also JP4.1
Changed lines of the file:
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@@
 <part name="GND9" library="SparkFun" deviceset="GND" device=""/>
 <part name="U$3" library="ondraster" deviceset="MICROUSB" device=""/>
+<part name="P+1" library="SparkFun" deviceset="VCC" device=""/>
 </parts>
 <sheets>
@@
 <instance part="GND9" gate="1" x="7.62" y="27.94"/>
 <instance part="U$3" gate="G$1" x="43.18" y="17.78"/>
+<instance part="P+1" gate="1" x="119.38" y="15.24"/>
 </instances>
 <busses>
@@
 <pinref part="P+3" gate="1" pin="VCC"/>
 </segment>
+<segment>
+<pinref part="JP4" gate="A" pin="1"/>
+<pinref part="P+1" gate="1" pin="VCC"/>
+<wire x1="119.38" y1="15.24" x2="121.92" y2="15.24" width="0.1524" layer="91"/>
+</segment>
 </net>
 <net name="/RST" class="0">
@@
 <junction x="25.4" y="-17.78"/>
 </segment>
-<segment>
-<wire x1="121.92" y1="15.24" x2="116.84" y2="15.24" width="0.1524" layer="91"/>
-<label x="116.84" y="15.24" size="1.778" layer="95"/>
-<pinref part="JP4" gate="A" pin="1"/>
-</segment>
-</net>
+</net>
