File: schematics/motorplank/motorplank.brd (EAGLE design)
At the start: 80 x 49 mm, 18 parts, among them IC1 74AHC1G86DBV

Commit message: Layout tweaks to motor plank.
Parts:
- R1, R2: value (none) -> 900
Changed lines of the file:
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@@
 <element name="U$5" library="nickparts" package="BILED" value="BILED" x="6.6675" y="35.8775"/>
 <element name="U$6" library="nickparts" package="BILED" value="BILED" x="6.35" y="13.0175"/>
-<element name="R1" library="SparkFun-Passives" package="0805" value="" x="6.6675" y="33.3375"/>
-<element name="R2" library="SparkFun-Passives" package="0805" value="" x="6.35" y="15.5575" rot="R180"/>
+<element name="R1" library="SparkFun-Passives" package="0805" value="900" x="6.6675" y="33.3375"/>
+<element name="R2" library="SparkFun-Passives" package="0805" value="900" x="6.35" y="15.5575" rot="R180"/>
 </elements>
 <signals>
