File: schematics/protoplank/protoplank.sch (EAGLE design)
At the start: 111 parts, among them IC1 74AHC1G86DBV

Commit message: Fix write protect pullups on plank EEPROMs.
Connections:
- net +3V3: now also WP.2
- net GND: no longer WP.2
Changed lines of the file:
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@@
 <part name="GND3" library="supply1" deviceset="GND" device=""/>
 <part name="WP" library="jumper" deviceset="SJ" device=""/>
-<part name="GND4" library="supply1" deviceset="GND" device=""/>
 <part name="U$3" library="nickparts" deviceset="PROTOPAD-3" device=""/>
 <part name="U$4" library="nickparts" deviceset="PROTOPAD-3" device=""/>
@@
 <instance part="P+2" gate="1" x="25.4" y="40.64"/>
 <instance part="U$2" gate="G$1" x="58.42" y="27.94"/>
-<instance part="+3V3" gate="G$1" x="71.12" y="35.56"/>
+<instance part="+3V3" gate="G$1" x="91.44" y="35.56"/>
 <instance part="GND3" gate="1" x="45.72" y="22.86"/>
 <instance part="WP" gate="1" x="81.28" y="30.48"/>
-<instance part="GND4" gate="1" x="86.36" y="25.4"/>
 <instance part="U$3" gate="G$1" x="200.66" y="121.92"/>
 <instance part="U$4" gate="G$1" x="205.74" y="121.92"/>
@@
 <pinref part="U$2" gate="G$1" pin="VCC"/>
 <pinref part="+3V3" gate="G$1" pin="+3V3"/>
+<wire x1="91.44" y1="33.02" x2="71.12" y2="33.02" width="0.1524" layer="91"/>
+<pinref part="WP" gate="1" pin="2"/>
+<wire x1="86.36" y1="30.48" x2="91.44" y2="30.48" width="0.1524" layer="91"/>
+<wire x1="91.44" y1="30.48" x2="91.44" y2="33.02" width="0.1524" layer="91"/>
+<junction x="91.44" y="33.02"/>
 </segment>
 <segment>
@@
 </segment>
 <segment>
-<pinref part="WP" gate="1" pin="2"/>
-<pinref part="GND4" gate="1" pin="GND"/>
-<wire x1="86.36" y1="30.48" x2="86.36" y2="27.94" width="0.1524" layer="91"/>
-</segment>
-<segment>
