File: schematics/soundplank/soundplank.sch (EAGLE design)
At the start: 19 parts, among them IC1 74AHC1G86DBV

Commit message: Updated soundplank to make use of opamp outputs when on the bottom.
Connections:
- removed net N$10 (its old number): U$1I1.7, U$1O1.4
- removed net N$11 (its old number): U$1I1.6, U$1O1.3
- removed net N$12 (its old number): U$1I1.5, U$1O1.2
- removed net N$13 (its old number): U$1I1.4, U$1O1.1
- removed net N$9 (its old number): U$1I1.8, U$1O1.5
- new net N$1: U$1I1.2, U$1O1.1
- new net N$2: U$1I1.3, U$1O1.2
- new net N$3: U$1I1.4, U$1O1.3
- new net N$4: U$1I1.5, U$1O1.4
- new net N$5: U$1I1.6, U$1O1.5
- net INL: now also U$1I2.2; no longer U$1I1.1
- net INR: now also U$1I2.1; no longer U$1I1.2
- net IR: now also U$1I2.3; no longer U$1I1.3
- net OUTL: now also U$1I1.8; no longer U$1I2.1
- net OUTR: now also U$1I1.7; no longer U$1I2.2
- net VOL: now also U$1I1.1; no longer U$1I2.3
Other:
- moved on the sheet: U$1O1

Commit message: Fix footprints on the soundplank so they're not backwards (oops!)
Connections:
- net INL: now also U$1I2.1; no longer U$1I2.2
- net INR: now also U$1I2.2; no longer U$1I2.1
- net OUTL: now also U$1I1.7; no longer U$1I1.8
- net OUTR: now also U$1I1.8; no longer U$1I1.7
Changed lines of the file:
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@@
 </segment>
 <segment>
-<pinref part="U$1" gate="I1" pin="8"/>
-<wire x1="7.62" y1="88.9" x2="10.16" y2="88.9" width="0.1524" layer="91"/>
-<label x="7.62" y="88.9" size="1.778" layer="95"/>
+<pinref part="U$1" gate="I1" pin="7"/>
+<wire x1="7.62" y1="91.44" x2="10.16" y2="91.44" width="0.1524" layer="91"/>
+<label x="7.62" y="91.44" size="1.778" layer="95"/>
 </segment>
 </net>
@@
 </segment>
 <segment>
-<pinref part="U$1" gate="I1" pin="7"/>
-<wire x1="7.62" y1="91.44" x2="10.16" y2="91.44" width="0.1524" layer="91"/>
-<label x="7.62" y="91.44" size="1.778" layer="95"/>
+<pinref part="U$1" gate="I1" pin="8"/>
+<wire x1="7.62" y1="88.9" x2="10.16" y2="88.9" width="0.1524" layer="91"/>
+<label x="7.62" y="88.9" size="1.778" layer="95"/>
 </segment>
 </net>
@@
 </segment>
 <segment>
-<pinref part="U$1" gate="I2" pin="2"/>
-<wire x1="43.18" y1="104.14" x2="48.26" y2="104.14" width="0.1524" layer="91"/>
-<label x="45.72" y="104.14" size="1.778" layer="95"/>
+<pinref part="U$1" gate="I2" pin="1"/>
+<wire x1="43.18" y1="106.68" x2="48.26" y2="106.68" width="0.1524" layer="91"/>
+<label x="45.72" y="106.68" size="1.778" layer="95"/>
 </segment>
 </net>
@@
 </segment>
 <segment>
-<pinref part="U$1" gate="I2" pin="1"/>
-<wire x1="43.18" y1="106.68" x2="48.26" y2="106.68" width="0.1524" layer="91"/>
-<label x="45.72" y="106.68" size="1.778" layer="95"/>
+<pinref part="U$1" gate="I2" pin="2"/>
+<wire x1="43.18" y1="104.14" x2="48.26" y2="104.14" width="0.1524" layer="91"/>
+<label x="45.72" y="104.14" size="1.778" layer="95"/>
 </segment>
 </net>

Commit message: Fix write protect pullups on plank EEPROMs.
Connections:
- net +3V3: now also SJ1.2
- net GND: no longer SJ1.2
Changed lines of the file:
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@@
 <part name="GND3" library="supply1" deviceset="GND" device=""/>
 <part name="SJ1" library="jumper" deviceset="SJ" device=""/>
-<part name="GND4" library="supply1" deviceset="GND" device=""/>
 <part name="U$3" library="SparkFun-Connectors" deviceset="AUDIO-JACK2" device="PTH"/>
 <part name="U1" library="SparkFun-Connectors" deviceset="AUDIO-JACK" device="PTH"/>
@@
 <instance part="P+2" gate="1" x="25.4" y="40.64"/>
 <instance part="U$2" gate="G$1" x="58.42" y="27.94"/>
-<instance part="+3V3" gate="G$1" x="71.12" y="35.56"/>
+<instance part="+3V3" gate="G$1" x="91.44" y="35.56"/>
 <instance part="GND3" gate="1" x="45.72" y="22.86"/>
 <instance part="SJ1" gate="1" x="81.28" y="30.48"/>
-<instance part="GND4" gate="1" x="86.36" y="25.4"/>
 <instance part="U$3" gate="G$1" x="99.06" y="63.5" smashed="yes" rot="MR180">
 <attribute name="NAME" x="93.98" y="57.912" size="1.778" layer="95" rot="MR180"/>
@@
 <pinref part="U$2" gate="G$1" pin="VCC"/>
 <pinref part="+3V3" gate="G$1" pin="+3V3"/>
+<wire x1="91.44" y1="33.02" x2="71.12" y2="33.02" width="0.1524" layer="91"/>
+<pinref part="SJ1" gate="1" pin="2"/>
+<wire x1="86.36" y1="30.48" x2="91.44" y2="30.48" width="0.1524" layer="91"/>
+<wire x1="91.44" y1="30.48" x2="91.44" y2="33.02" width="0.1524" layer="91"/>
+<junction x="91.44" y="33.02"/>
 </segment>
 <segment>
@@
 </segment>
 <segment>
-<pinref part="SJ1" gate="1" pin="2"/>
-<pinref part="GND4" gate="1" pin="GND"/>
-<wire x1="86.36" y1="30.48" x2="86.36" y2="27.94" width="0.1524" layer="91"/>
-</segment>
-<segment>
